Commit message: robot_in_gazebo

File: description/robot_core.xacro (robot description, xacro)
@@ -39,4 +39,5 @@
         </xacro:inertial_box>
     </link>
+    <gazebo reference="chassis"> <material>Gazebo/Orange</material></gazebo>
     <joint name="left_wheel_joint" type="continuous">
         <origin xyz="0 0.175 0" rpy="${pi/2} 0 0"></origin>
@@ -62,4 +63,5 @@
         </xacro:inertial_cylinder>
     </link>
+        <gazebo reference="left_wheel"> <material>Gazebo/Black</material></gazebo>
     <joint name="right_wheel_joint" type="continuous">
         <origin xyz="0 -0.175 0" rpy="${pi/2} 0 0"></origin>
@@ -85,4 +87,5 @@
         </xacro:inertial_cylinder>
     </link>
+        <gazebo reference="right_wheel"> <material>Gazebo/Black</material></gazebo>
     <joint name="caster_wheel_joint" type="fixed">
         <origin xyz="0.25 0 0"></origin>
@@ -107,3 +110,8 @@
         </xacro:inertial_sphere>
     </link>
+        <gazebo reference="caster_wheel">
+            <material>Gazebo/White</material>
+            <mu1 value="0.001"></mu1>
+            <mu2 value="0.001"></mu2>
+        </gazebo>
 </robot>
